File: ethernet.sch (KiCad schematic (older format))
At the start: 32 parts, among them J3 L834-1G1T-91, U9 LAN8742A, Y3 25M

Commit message: Replace non stocked components.
 - Redesign 5V/3.3V using TPS6216xDSGT
 - Use bigger crystal (move to 5031 case)
 - Change some components parts

Signed-off-by: Martin Ribelotta <martinribelotta@gmail.com>
Parts:
- C25, C29: DESCRIPTION (none) -> Capacitor 10p 0603
- C30, C36: DESCRIPTION (none) -> Capacitor 10u 0603
- C31, C33, C35: DESCRIPTION (none) -> Capacitor 100n 0603
- C32: value 420p -> 470p; DESCRIPTION (none) -> Capacitor 420p 0603
- C34: DESCRIPTION (none) -> Capacitor 1u 0603
- C37, C38: DESCRIPTION (none) -> Capacitor 0.022u 0603
- L5: DESCRIPTION (none) -> ferrite bead 0603
- R10, R11, R12, R8: DESCRIPTION (none) -> Resistor 49.9 ohm 1%0603
- R13, R14, R15, R16, R17, R18, R22, R6, R7: DESCRIPTION (none) -> Resistor 10K 0603
- R19: DESCRIPTION (none) -> Resistor 1.5K 0603
- R24, R25: DESCRIPTION (none) -> Resistor 270 ohm 0603
- R9: DESCRIPTION (none) -> Resistor 12.1K 1% 0603
- U9: DESCRIPTION (none) -> LAN8742A
- Y3: footprint footprints:Crystal_SMD_3215-2Pin_3.2x1.5mm -> Crystal:Crystal_SMD_5032-2Pin_5.0x3.2mm; DESCRIPTION (none) -> Crystal 25MHz 3215
Changed lines of the file:
@@
 F 29 "+70°C" H 4600 7100 50  0001 L CNN "temperature range high"
 F 30 "0°C" H 4600 7200 50  0001 L CNN "temperature range low"
+F 31 "LAN8742A" H 4600 4000 50  0001 C CNN "DESCRIPTION"
 	1    4600 4000
 	1    0    0    -1
@@
 F 2 "Capacitor_SMD:C_0603_1608Metric" H 7400 4600 50  0001 C CNN
 F 3 "~" H 7400 4600 50  0001 C CNN
+F 4 "Capacitor 0.022u 0603" H 7400 4600 50  0001 C CNN "DESCRIPTION"
 	1    7400 4600
 	1    0    0    -1
@@
 F 2 "Resistor_SMD:R_0603_1608Metric" H 5700 3200 50  0001 C CNN
 F 3 "~" H 5700 3200 50  0001 C CNN
+F 4 "Resistor 49.9 ohm 1%0603" H 5700 3200 50  0001 C CNN "DESCRIPTION"
 	1    5700 3200
 	1    0    0    -1
@@
 F 2 "Resistor_SMD:R_0603_1608Metric" H 6050 3200 50  0001 C CNN
 F 3 "~" H 6050 3200 50  0001 C CNN
+F 4 "Resistor 49.9 ohm 1%0603" H 6050 3200 50  0001 C CNN "DESCRIPTION"
 	1    6050 3200
 	1    0    0    -1
@@
 F 2 "Resistor_SMD:R_0603_1608Metric" H 6400 3200 50  0001 C CNN
 F 3 "~" H 6400 3200 50  0001 C CNN
+F 4 "Resistor 49.9 ohm 1%0603" H 6400 3200 50  0001 C CNN "DESCRIPTION"
 	1    6400 3200
 	1    0    0    -1
@@
 F 2 "Resistor_SMD:R_0603_1608Metric" H 6750 3200 50  0001 C CNN
 F 3 "~" H 6750 3200 50  0001 C CNN
+F 4 "Resistor 49.9 ohm 1%0603" H 6750 3200 50  0001 C CNN "DESCRIPTION"
 	1    6750 3200
 	1    0    0    -1
@@
 F 2 "Capacitor_SMD:C_0603_1608Metric" H 4950 2800 50  0001 C CNN
 F 3 "~" H 4950 2800 50  0001 C CNN
+F 4 "Capacitor 100n 0603" H 4950 2800 50  0001 C CNN "DESCRIPTION"
 	1    4950 2800
 	1    0    0    -1
@@
 AR Path="/60185BCA/601E973F" Ref="C32"  Part="1"
 F 0 "C32" H 5042 2496 50  0000 L CNN
-F 1 "420p" H 5042 2405 50  0000 L CNN
+F 1 "470p" H 5042 2405 50  0000 L CNN
 F 2 "Capacitor_SMD:C_0603_1608Metric" H 4950 2450 50  0001 C CNN
 F 3 "~" H 4950 2450 50  0001 C CNN
+F 4 "Capacitor 420p 0603" H 4950 2450 50  0001 C CNN "DESCRIPTION"
 	1    4950 2450
 	1    0    0    -1
@@
 F 2 "Capacitor_SMD:C_0603_1608Metric" H 5300 2450 50  0001 C CNN
 F 3 "~" H 5300 2450 50  0001 C CNN
+F 4 "Capacitor 1u 0603" H 5300 2450 50  0001 C CNN "DESCRIPTION"
 	1    5300 2450
 	1    0    0    -1
@@
 F 2 "Capacitor_SMD:C_0603_1608Metric" H 5650 2800 50  0001 C CNN
 F 3 "~" H 5650 2800 50  0001 C CNN
+F 4 "Capacitor 10u 0603" H 5650 2800 50  0001 C CNN "DESCRIPTION"
 	1    5650 2800
 	1    0    0    -1
@@
 F 2 "Capacitor_SMD:C_0603_1608Metric" H 5300 2800 50  0001 C CNN
 F 3 "~" H 5300 2800 50  0001 C CNN
+F 4 "Capacitor 100n 0603" H 5300 2800 50  0001 C CNN "DESCRIPTION"
 	1    5300 2800
 	1    0    0    -1
@@
 F 2 "Capacitor_SMD:C_0603_1608Metric" H 3650 2800 50  0001 C CNN
 F 3 "~" H 3650 2800 50  0001 C CNN
+F 4 "Capacitor 10u 0603" H 3650 2800 50  0001 C CNN "DESCRIPTION"
 	1    3650 2800
 	-1   0    0    -1
@@
 F 2 "Capacitor_SMD:C_0603_1608Metric" H 4050 2800 50  0001 C CNN
 F 3 "~" H 4050 2800 50  0001 C CNN
+F 4 "Capacitor 100n 0603" H 4050 2800 50  0001 C CNN "DESCRIPTION"
 	1    4050 2800
 	-1   0    0    -1
@@
 F 2 "Inductor_SMD:L_0603_1608Metric" H 4400 2700 50  0001 C CNN
 F 3 "~" H 4400 2700 50  0001 C CNN
+F 4 "ferrite bead 0603" H 4400 2700 50  0001 C CNN "DESCRIPTION"
 	1    4400 2700
 	0    -1   -1   0
@@
 F 2 "Resistor_SMD:R_0603_1608Metric" H 5350 4600 50  0001 C CNN
 F 3 "~" H 5350 4600 50  0001 C CNN
+F 4 "Resistor 12.1K 1% 0603" H 5350 4600 50  0001 C CNN "DESCRIPTION"
 	1    5350 4600
 	1    0    0    -1
@@
 F 2 "Capacitor_SMD:C_0603_1608Metric" H 3600 4950 50  0001 C CNN
 F 3 "~" H 3600 4950 50  0001 C CNN
+F 4 "Capacitor 10p 0603" H 3600 4950 50  0001 C CNN "DESCRIPTION"
 	1    3600 4950
 	1    0    0    1
@@
 F 2 "Capacitor_SMD:C_0603_1608Metric" H 3200 4950 50  0001 C CNN
 F 3 "~" H 3200 4950 50  0001 C CNN
+F 4 "Capacitor 10p 0603" H 3200 4950 50  0001 C CNN "DESCRIPTION"
 	1    3200 4950
 	1    0    0    1
@@
 F 0 "Y3" H 3400 4925 50  0000 C CNN
 F 1 "25M" H 3400 4834 50  0000 C CNN
-F 2 "footprints:Crystal_SMD_3215-2Pin_3.2x1.5mm" H 3400 4700 50  0001 C CNN
+F 2 "Crystal:Crystal_SMD_5032-2Pin_5.0x3.2mm" H 3400 4700 50  0001 C CNN
 F 3 "~" H 3400 4700 50  0001 C CNN
+F 4 "Crystal 25MHz 3215" H 3400 4700 50  0001 C CNN "DESCRIPTION"
 	1    3400 4700
 	1    0    0    1
@@
 F 2 "Resistor_SMD:R_0603_1608Metric" H 5850 4600 50  0001 C CNN
 F 3 "~" H 5850 4600 50  0001 C CNN
+F 4 "Resistor 10K 0603" H 5850 4600 50  0001 C CNN "DESCRIPTION"
 	1    5850 4600
 	-1   0    0    1
@@
 F 2 "Capacitor_SMD:C_0603_1608Metric" H 6950 4600 50  0001 C CNN
 F 3 "~" H 6950 4600 50  0001 C CNN
+F 4 "Capacitor 0.022u 0603" H 6950 4600 50  0001 C CNN "DESCRIPTION"
 	1    6950 4600
 	-1   0    0    -1
@@
 F 2 "Resistor_SMD:R_0603_1608Metric" H 6800 4350 50  0001 C CNN
 F 3 "~" H 6800 4350 50  0001 C CNN
+F 4 "Resistor 270 ohm 0603" H 6800 4350 50  0001 C CNN "DESCRIPTION"
 	1    6800 4350
 	0    -1   -1   0
@@
 F 2 "Resistor_SMD:R_0603_1608Metric" H 6800 4150 50  0001 C CNN
 F 3 "~" H 6800 4150 50  0001 C CNN
+F 4 "Resistor 270 ohm 0603" H 6800 4150 50  0001 C CNN "DESCRIPTION"
 	1    6800 4150
 	0    -1   -1   0
@@
 F 2 "Resistor_SMD:R_0603_1608Metric" H 1650 3950 50  0001 C CNN
 F 3 "~" H 1650 3950 50  0001 C CNN
+F 4 "Resistor 10K 0603" H 1650 3950 50  0001 C CNN "DESCRIPTION"
 	1    1650 3950
 	0    -1   -1   0
@@
 F 2 "Resistor_SMD:R_0603_1608Metric" H 2750 3250 50  0001 C CNN
 F 3 "~" H 2750 3250 50  0001 C CNN
+F 4 "Resistor 10K 0603" H 2750 3250 50  0001 C CNN "DESCRIPTION"
 	1    2750 3250
 	1    0    0    -1
@@
 F 2 "Resistor_SMD:R_0603_1608Metric" H 3050 3250 50  0001 C CNN
 F 3 "~" H 3050 3250 50  0001 C CNN
+F 4 "Resistor 10K 0603" H 3050 3250 50  0001 C CNN "DESCRIPTION"
 	1    3050 3250
 	1    0    0    -1
@@
 F 2 "Resistor_SMD:R_0603_1608Metric" H 3350 3250 50  0001 C CNN
 F 3 "~" H 3350 3250 50  0001 C CNN
+F 4 "Resistor 10K 0603" H 3350 3250 50  0001 C CNN "DESCRIPTION"
 	1    3350 3250
 	1    0    0    -1
@@
 F 2 "Resistor_SMD:R_0603_1608Metric" H 3650 3250 50  0001 C CNN
 F 3 "~" H 3650 3250 50  0001 C CNN
+F 4 "Resistor 1.5K 0603" H 3650 3250 50  0001 C CNN "DESCRIPTION"
 	1    3650 3250
 	1    0    0    -1
@@
 F 2 "Resistor_SMD:R_0603_1608Metric" H 2500 3750 50  0001 C CNN
 F 3 "~" H 2500 3750 50  0001 C CNN
+F 4 "Resistor 10K 0603" H 2500 3750 50  0001 C CNN "DESCRIPTION"
 	1    2500 3750
 	0    1    1    0
@@
 F 2 "Resistor_SMD:R_0603_1608Metric" H 2500 3850 50  0001 C CNN
 F 3 "~" H 2500 3850 50  0001 C CNN
+F 4 "Resistor 10K 0603" H 2500 3850 50  0001 C CNN "DESCRIPTION"
 	1    2500 3850
 	0    1    1    0
@@
 F 2 "Resistor_SMD:R_0603_1608Metric" H 2500 4050 50  0001 C CNN
 F 3 "~" H 2500 4050 50  0001 C CNN
+F 4 "Resistor 10K 0603" H 2500 4050 50  0001 C CNN "DESCRIPTION"
 	1    2500 4050
 	0    1    -1   0
@@
 F 2 "Resistor_SMD:R_0603_1608Metric" H 2500 4450 50  0001 C CNN
 F 3 "~" H 2500 4450 50  0001 C CNN
+F 4 "Resistor 10K 0603" H 2500 4450 50  0001 C CNN "DESCRIPTION"
 	1    2500 4450
 	0    1    -1   0

Commit message: Add new BOM to octopart
TODO: PSRAM is not recognized by Octopart but is available in LCSC

Signed-off-by: Martin Ribelotta <martinribelotta@gmail.com>
Parts:
- C25, C29: MANUFACTURER (none) -> Yageo; MANUFACTURER_PART_NUMBER (none) -> CC0603JRNPO9BN100
- C30, C36: MANUFACTURER (none) -> AVX; MANUFACTURER_PART_NUMBER (none) -> 0603ZD106KAT2A
- C31, C33, C35: MANUFACTURER (none) -> Yageo; MANUFACTURER_PART_NUMBER (none) -> CC0603KRX7R9BB104
- C32: MANUFACTURER (none) -> AVX; MANUFACTURER_PART_NUMBER (none) -> 06035C471KAT2A
- C34: MANUFACTURER (none) -> Yageo; MANUFACTURER_PART_NUMBER (none) -> CC0603ZRY5V6BB105
- C37, C38: MANUFACTURER (none) -> AVX; MANUFACTURER_PART_NUMBER (none) -> 06035C223KAT2A
- J3: MANUFACTURER_PART_NUMBER (none) -> L834-1G1T-91
- L5: MANUFACTURER (none) -> Taiyo Yuden; MANUFACTURER_PART_NUMBER (none) -> BK1608HS220-T
- R10, R11, R12, R8: MANUFACTURER (none) -> Yageo; MANUFACTURER_PART_NUMBER (none) -> RC0603FR-0749R9L
- R13, R14, R15, R16, R17, R18, R22, R6, R7: MANUFACTURER (none) -> Yageo; MANUFACTURER_PART_NUMBER (none) -> RC0603FR-0710KL
- R19: MANUFACTURER (none) -> Yageo; MANUFACTURER_PART_NUMBER (none) -> RC0603JR-071K5L
- R24, R25: value 270R -> 220R; MANUFACTURER (none) -> Yageo; MANUFACTURER_PART_NUMBER (none) -> RC0603JR-07220RL
- R9: MANUFACTURER (none) -> Yageo; MANUFACTURER_PART_NUMBER (none) -> RT0603BRD0712K1L
- U9: MANUFACTURER (none) -> Microchip; MANUFACTURER_PART_NUMBER (none) -> LAN8742A
- Y3: MANUFACTURER (none) -> QST; MANUFACTURER_PART_NUMBER (none) -> QT3C-32.768KDZF-T
Changed lines of the file:
@@
 F 30 "0°C" H 4600 7200 50  0001 L CNN "temperature range low"
 F 31 "LAN8742A" H 4600 4000 50  0001 C CNN "DESCRIPTION"
+F 32 "Microchip" H 4600 4000 50  0001 C CNN "MANUFACTURER"
+F 33 "LAN8742A" H 4600 4000 50  0001 C CNN "MANUFACTURER_PART_NUMBER"
 	1    4600 4000
 	1    0    0    -1
@@
 F 3 "~" H 7400 4600 50  0001 C CNN
 F 4 "Capacitor 0.022u 0603" H 7400 4600 50  0001 C CNN "DESCRIPTION"
+F 5 "AVX" H 7400 4600 50  0001 C CNN "MANUFACTURER"
+F 6 "06035C223KAT2A" H 7400 4600 50  0001 C CNN "MANUFACTURER_PART_NUMBER"
 	1    7400 4600
 	1    0    0    -1
@@
 F 3 "~" H 5700 3200 50  0001 C CNN
 F 4 "Resistor 49.9 ohm 1%0603" H 5700 3200 50  0001 C CNN "DESCRIPTION"
+F 5 "Yageo" H 5700 3200 50  0001 C CNN "MANUFACTURER"
+F 6 "RC0603FR-0749R9L" H 5700 3200 50  0001 C CNN "MANUFACTURER_PART_NUMBER"
 	1    5700 3200
 	1    0    0    -1
@@
 F 3 "~" H 6050 3200 50  0001 C CNN
 F 4 "Resistor 49.9 ohm 1%0603" H 6050 3200 50  0001 C CNN "DESCRIPTION"
+F 5 "Yageo" H 6050 3200 50  0001 C CNN "MANUFACTURER"
+F 6 "RC0603FR-0749R9L" H 6050 3200 50  0001 C CNN "MANUFACTURER_PART_NUMBER"
 	1    6050 3200
 	1    0    0    -1
@@
 F 3 "~" H 6400 3200 50  0001 C CNN
 F 4 "Resistor 49.9 ohm 1%0603" H 6400 3200 50  0001 C CNN "DESCRIPTION"
+F 5 "Yageo" H 6400 3200 50  0001 C CNN "MANUFACTURER"
+F 6 "RC0603FR-0749R9L" H 6400 3200 50  0001 C CNN "MANUFACTURER_PART_NUMBER"
 	1    6400 3200
 	1    0    0    -1
@@
 F 3 "~" H 6750 3200 50  0001 C CNN
 F 4 "Resistor 49.9 ohm 1%0603" H 6750 3200 50  0001 C CNN "DESCRIPTION"
+F 5 "Yageo" H 6750 3200 50  0001 C CNN "MANUFACTURER"
+F 6 "RC0603FR-0749R9L" H 6750 3200 50  0001 C CNN "MANUFACTURER_PART_NUMBER"
 	1    6750 3200
 	1    0    0    -1
@@
 F 3 "~" H 4950 2800 50  0001 C CNN
 F 4 "Capacitor 100n 0603" H 4950 2800 50  0001 C CNN "DESCRIPTION"
+F 5 "CC0603KRX7R9BB104" H 4950 2800 50  0001 C CNN "MANUFACTURER_PART_NUMBER"
+F 6 "Yageo" H 4950 2800 50  0001 C CNN "MANUFACTURER"
 	1    4950 2800
 	1    0    0    -1
@@
 F 3 "~" H 4950 2450 50  0001 C CNN
 F 4 "Capacitor 420p 0603" H 4950 2450 50  0001 C CNN "DESCRIPTION"
+F 5 "AVX" H 4950 2450 50  0001 C CNN "MANUFACTURER"
+F 6 "06035C471KAT2A" H 4950 2450 50  0001 C CNN "MANUFACTURER_PART_NUMBER"
 	1    4950 2450
 	1    0    0    -1
@@
 F 3 "~" H 5300 2450 50  0001 C CNN
 F 4 "Capacitor 1u 0603" H 5300 2450 50  0001 C CNN "DESCRIPTION"
+F 5 "CC0603ZRY5V6BB105" H 5300 2450 50  0001 C CNN "MANUFACTURER_PART_NUMBER"
+F 6 "Yageo" H 5300 2450 50  0001 C CNN "MANUFACTURER"
 	1    5300 2450
 	1    0    0    -1
@@
 F 3 "~" H 5650 2800 50  0001 C CNN
 F 4 "Capacitor 10u 0603" H 5650 2800 50  0001 C CNN "DESCRIPTION"
+F 5 "AVX" H 5650 2800 50  0001 C CNN "MANUFACTURER"
+F 6 "0603ZD106KAT2A" H 5650 2800 50  0001 C CNN "MANUFACTURER_PART_NUMBER"
 	1    5650 2800
 	1    0    0    -1
@@
 F 3 "~" H 5300 2800 50  0001 C CNN
 F 4 "Capacitor 100n 0603" H 5300 2800 50  0001 C CNN "DESCRIPTION"
+F 5 "CC0603KRX7R9BB104" H 5300 2800 50  0001 C CNN "MANUFACTURER_PART_NUMBER"
+F 6 "Yageo" H 5300 2800 50  0001 C CNN "MANUFACTURER"
 	1    5300 2800
 	1    0    0    -1
@@
 F 3 "~" H 3650 2800 50  0001 C CNN
 F 4 "Capacitor 10u 0603" H 3650 2800 50  0001 C CNN "DESCRIPTION"
+F 5 "AVX" H 3650 2800 50  0001 C CNN "MANUFACTURER"
+F 6 "0603ZD106KAT2A" H 3650 2800 50  0001 C CNN "MANUFACTURER_PART_NUMBER"
 	1    3650 2800
 	-1   0    0    -1
@@
 F 3 "~" H 4050 2800 50  0001 C CNN
 F 4 "Capacitor 100n 0603" H 4050 2800 50  0001 C CNN "DESCRIPTION"
+F 5 "CC0603KRX7R9BB104" H 4050 2800 50  0001 C CNN "MANUFACTURER_PART_NUMBER"
+F 6 "Yageo" H 4050 2800 50  0001 C CNN "MANUFACTURER"
 	1    4050 2800
 	-1   0    0    -1
@@
 F 3 "~" H 4400 2700 50  0001 C CNN
 F 4 "ferrite bead 0603" H 4400 2700 50  0001 C CNN "DESCRIPTION"
+F 5 "Taiyo Yuden" H 4400 2700 50  0001 C CNN "MANUFACTURER"
+F 6 "BK1608HS220-T" H 4400 2700 50  0001 C CNN "MANUFACTURER_PART_NUMBER"
 	1    4400 2700
 	0    -1   -1   0
@@
 F 3 "~" H 5350 4600 50  0001 C CNN
 F 4 "Resistor 12.1K 1% 0603" H 5350 4600 50  0001 C CNN "DESCRIPTION"
+F 5 "Yageo" H 5350 4600 50  0001 C CNN "MANUFACTURER"
+F 6 "RT0603BRD0712K1L" H 5350 4600 50  0001 C CNN "MANUFACTURER_PART_NUMBER"
 	1    5350 4600
 	1    0    0    -1
@@
 F 3 "~" H 3600 4950 50  0001 C CNN
 F 4 "Capacitor 10p 0603" H 3600 4950 50  0001 C CNN "DESCRIPTION"
+F 5 "CC0603JRNPO9BN100" H 3600 4950 50  0001 C CNN "MANUFACTURER_PART_NUMBER"
+F 6 "Yageo" H 3600 4950 50  0001 C CNN "MANUFACTURER"
 	1    3600 4950
 	1    0    0    1
@@
 F 3 "~" H 3200 4950 50  0001 C CNN
 F 4 "Capacitor 10p 0603" H 3200 4950 50  0001 C CNN "DESCRIPTION"
+F 5 "CC0603JRNPO9BN100" H 3200 4950 50  0001 C CNN "MANUFACTURER_PART_NUMBER"
+F 6 "Yageo" H 3200 4950 50  0001 C CNN "MANUFACTURER"
 	1    3200 4950
 	1    0    0    1
@@
 F 3 "~" H 3400 4700 50  0001 C CNN
 F 4 "Crystal 25MHz 3215" H 3400 4700 50  0001 C CNN "DESCRIPTION"
+F 5 "QST" H 3400 4700 50  0001 C CNN "MANUFACTURER"
+F 6 "QT3C-32.768KDZF-T" H 3400 4700 50  0001 C CNN "MANUFACTURER_PART_NUMBER"
 	1    3400 4700
 	1    0    0    1
@@
 F 3 "~" H 5850 4600 50  0001 C CNN
 F 4 "Resistor 10K 0603" H 5850 4600 50  0001 C CNN "DESCRIPTION"
+F 5 "Yageo" H 5850 4600 50  0001 C CNN "MANUFACTURER"
+F 6 "RC0603FR-0710KL" H 5850 4600 50  0001 C CNN "MANUFACTURER_PART_NUMBER"
 	1    5850 4600
 	-1   0    0    1
@@
 F 3 "~" H 6950 4600 50  0001 C CNN
 F 4 "Capacitor 0.022u 0603" H 6950 4600 50  0001 C CNN "DESCRIPTION"
+F 5 "AVX" H 6950 4600 50  0001 C CNN "MANUFACTURER"
+F 6 "06035C223KAT2A" H 6950 4600 50  0001 C CNN "MANUFACTURER_PART_NUMBER"
 	1    6950 4600
 	-1   0    0    -1
@@
 AR Path="/60185BCA/60577D04" Ref="R25"  Part="1"
 F 0 "R25" V 6850 3950 50  0000 C CNN
-F 1 "270R" V 6850 4150 50  0000 C CNN
+F 1 "220R" V 6850 4150 50  0000 C CNN
 F 2 "Resistor_SMD:R_0603_1608Metric" H 6800 4350 50  0001 C CNN
 F 3 "~" H 6800 4350 50  0001 C CNN
 F 4 "Resistor 270 ohm 0603" H 6800 4350 50  0001 C CNN "DESCRIPTION"
+F 5 "Yageo" H 6800 4350 50  0001 C CNN "MANUFACTURER"
+F 6 "RC0603JR-07220RL" H 6800 4350 50  0001 C CNN "MANUFACTURER_PART_NUMBER"
 	1    6800 4350
 	0    -1   -1   0
@@
 AR Path="/60185BCA/60588F84" Ref="R24"  Part="1"
 F 0 "R24" V 6850 3750 50  0000 C CNN
-F 1 "270R" V 6850 3950 50  0000 C CNN
+F 1 "220R" V 6850 3950 50  0000 C CNN
 F 2 "Resistor_SMD:R_0603_1608Metric" H 6800 4150 50  0001 C CNN
 F 3 "~" H 6800 4150 50  0001 C CNN
 F 4 "Resistor 270 ohm 0603" H 6800 4150 50  0001 C CNN "DESCRIPTION"
+F 5 "Yageo" H 6800 4150 50  0001 C CNN "MANUFACTURER"
+F 6 "RC0603JR-07220RL" H 6800 4150 50  0001 C CNN "MANUFACTURER_PART_NUMBER"
 	1    6800 4150
 	0    -1   -1   0
@@
 F 6 "C" H 8000 4050 50  0001 L BNN "PARTREV"
 F 7 "11.46 mm" H 8000 4050 50  0001 L BNN "MAXIMUM_PACKAGE_HEIGHT"
+F 8 "L834-1G1T-91" H 8000 4050 50  0001 C CNN "MANUFACTURER_PART_NUMBER"
 	1    8000 4050
 	1    0    0    -1
@@
 F 3 "~" H 1650 3950 50  0001 C CNN
 F 4 "Resistor 10K 0603" H 1650 3950 50  0001 C CNN "DESCRIPTION"
+F 5 "Yageo" H 1650 3950 50  0001 C CNN "MANUFACTURER"
+F 6 "RC0603FR-0710KL" H 1650 3950 50  0001 C CNN "MANUFACTURER_PART_NUMBER"
 	1    1650 3950
 	0    -1   -1   0
@@
 F 3 "~" H 2750 3250 50  0001 C CNN
 F 4 "Resistor 10K 0603" H 2750 3250 50  0001 C CNN "DESCRIPTION"
+F 5 "Yageo" H 2750 3250 50  0001 C CNN "MANUFACTURER"
+F 6 "RC0603FR-0710KL" H 2750 3250 50  0001 C CNN "MANUFACTURER_PART_NUMBER"
 	1    2750 3250
 	1    0    0    -1
@@
 F 3 "~" H 3050 3250 50  0001 C CNN
 F 4 "Resistor 10K 0603" H 3050 3250 50  0001 C CNN "DESCRIPTION"
+F 5 "Yageo" H 3050 3250 50  0001 C CNN "MANUFACTURER"
+F 6 "RC0603FR-0710KL" H 3050 3250 50  0001 C CNN "MANUFACTURER_PART_NUMBER"
 	1    3050 3250
 	1    0    0    -1
@@
 F 3 "~" H 3350 3250 50  0001 C CNN
 F 4 "Resistor 10K 0603" H 3350 3250 50  0001 C CNN "DESCRIPTION"
+F 5 "Yageo" H 3350 3250 50  0001 C CNN "MANUFACTURER"
+F 6 "RC0603FR-0710KL" H 3350 3250 50  0001 C CNN "MANUFACTURER_PART_NUMBER"
 	1    3350 3250
 	1    0    0    -1
@@
 F 3 "~" H 3650 3250 50  0001 C CNN
 F 4 "Resistor 1.5K 0603" H 3650 3250 50  0001 C CNN "DESCRIPTION"
+F 5 "Yageo" H 3650 3250 50  0001 C CNN "MANUFACTURER"
+F 6 "RC0603JR-071K5L" H 3650 3250 50  0001 C CNN "MANUFACTURER_PART_NUMBER"
 	1    3650 3250
 	1    0    0    -1
@@
 F 3 "~" H 2500 3750 50  0001 C CNN
 F 4 "Resistor 10K 0603" H 2500 3750 50  0001 C CNN "DESCRIPTION"
+F 5 "Yageo" H 2500 3750 50  0001 C CNN "MANUFACTURER"
+F 6 "RC0603FR-0710KL" H 2500 3750 50  0001 C CNN "MANUFACTURER_PART_NUMBER"
 	1    2500 3750
 	0    1    1    0
@@
 F 3 "~" H 2500 3850 50  0001 C CNN
 F 4 "Resistor 10K 0603" H 2500 3850 50  0001 C CNN "DESCRIPTION"
+F 5 "Yageo" H 2500 3850 50  0001 C CNN "MANUFACTURER"
+F 6 "RC0603FR-0710KL" H 2500 3850 50  0001 C CNN "MANUFACTURER_PART_NUMBER"
 	1    2500 3850
 	0    1    1    0
@@
 F 3 "~" H 2500 4050 50  0001 C CNN
 F 4 "Resistor 10K 0603" H 2500 4050 50  0001 C CNN "DESCRIPTION"
+F 5 "Yageo" H 2500 4050 50  0001 C CNN "MANUFACTURER"
+F 6 "RC0603FR-0710KL" H 2500 4050 50  0001 C CNN "MANUFACTURER_PART_NUMBER"
 	1    2500 4050
 	0    1    -1   0
@@
 F 3 "~" H 2500 4450 50  0001 C CNN
 F 4 "Resistor 10K 0603" H 2500 4450 50  0001 C CNN "DESCRIPTION"
+F 5 "Yageo" H 2500 4450 50  0001 C CNN "MANUFACTURER"
+F 6 "RC0603FR-0710KL" H 2500 4450 50  0001 C CNN "MANUFACTURER_PART_NUMBER"
 	1    2500 4450
 	0    1    -1   0

Commit message: Update schemas
Signed-off-by: Martin Ribelotta <martinribelotta@gmail.com>
Parts:
- Y3: MANUFACTURER QST -> Abracom; MANUFACTURER_PART_NUMBER QT3C-32.768KDZF-T -> ABM7-25.000MHZ-D2Y-T
Changed lines of the file:
@@
 F 3 "~" H 3400 4700 50  0001 C CNN
 F 4 "Crystal 25MHz 3215" H 3400 4700 50  0001 C CNN "DESCRIPTION"
-F 5 "QST" H 3400 4700 50  0001 C CNN "MANUFACTURER"
-F 6 "QT3C-32.768KDZF-T" H 3400 4700 50  0001 C CNN "MANUFACTURER_PART_NUMBER"
+F 5 "Abracom" H 3400 4700 50  0001 C CNN "MANUFACTURER"
+F 6 "ABM7-25.000MHZ-D2Y-T" H 3400 4700 50  0001 C CNN "MANUFACTURER_PART_NUMBER"
 	1    3400 4700
 	1    0    0    1
