File: ethernet.sch (KiCad schematic (older format))
At the start: 32 parts, among them J3 L834-1G1T-91, U9 LAN8742A, Y3 25M

Commit message: Prepare for send to PCBWay
Signed-off-by: Martin Ribelotta <martinribelotta@gmail.com>
Parts:
- J3: DESCRIPTION (none) -> L834-1G1T-91
Connections:
- net GND: now also R24.1; no longer J3.13
- net LED1: now also J3.14; no longer R24.1
- net at R24.2: now also J3.13; no longer J3.14
Other:
- moved on the sheet: R24
Changed lines of the file:
@@
 L Device:R_Small R?
 U 1 1 60588F84
-P 6800 4150
+P 6800 4250
 AR Path="/60588F84" Ref="R?"  Part="1"
 AR Path="/60185BCA/60588F84" Ref="R24"  Part="1"
-F 0 "R24" V 6850 3750 50  0000 C CNN
-F 1 "220R" V 6850 3950 50  0000 C CNN
-F 2 "Resistor_SMD:R_0603_1608Metric" H 6800 4150 50  0001 C CNN
-F 3 "~" H 6800 4150 50  0001 C CNN
-F 4 "Resistor 270 ohm 0603" H 6800 4150 50  0001 C CNN "DESCRIPTION"
-F 5 "Yageo" H 6800 4150 50  0001 C CNN "MANUFACTURER"
-F 6 "RC0603JR-07220RL" H 6800 4150 50  0001 C CNN "MANUFACTURER_PART_NUMBER"
-	1    6800 4150
+F 0 "R24" V 6850 3850 50  0000 C CNN
+F 1 "220R" V 6850 4050 50  0000 C CNN
+F 2 "Resistor_SMD:R_0603_1608Metric" H 6800 4250 50  0001 C CNN
+F 3 "~" H 6800 4250 50  0001 C CNN
+F 4 "Resistor 270 ohm 0603" H 6800 4250 50  0001 C CNN "DESCRIPTION"
+F 5 "Yageo" H 6800 4250 50  0001 C CNN "MANUFACTURER"
+F 6 "RC0603JR-07220RL" H 6800 4250 50  0001 C CNN "MANUFACTURER_PART_NUMBER"
+	1    6800 4250
 	0    -1   -1   0
 $EndComp
@@
 F 7 "11.46 mm" H 8000 4050 50  0001 L BNN "MAXIMUM_PACKAGE_HEIGHT"
 F 8 "L834-1G1T-91" H 8000 4050 50  0001 C CNN "MANUFACTURER_PART_NUMBER"
+F 9 "L834-1G1T-91" H 8000 4050 50  0001 C CNN "DESCRIPTION"
 	1    8000 4050
 	1    0    0    -1
@@
 Connection ~ 7500 4700
 Wire Wire Line
-	6900 4150 7500 4150
-Wire Wire Line
 	7500 4350 6900 4350
 Wire Wire Line
-	6550 4250 7500 4250
+	6550 4250 6700 4250
 Wire Wire Line
 	6550 4450 7500 4450
@@
 Wire Wire Line
 	5850 4700 6550 4700
-Wire Wire Line
-	5200 4150 6700 4150
 $Comp
 L Device:R_Small R?
@@
 	5900 2700 5650 2700
 Connection ~ 5650 2700
+Wire Wire Line
+	6900 4250 7500 4250
+Wire Wire Line
+	5200 4150 7500 4150
 $EndSCHEMATC
