File: h730duino.kicad_pcb (KiCad board)
At the start: 4 copper layers, 101.6 x 53.3 mm, 124 parts, among them J1 USB_C_Receptacle_USB2.0, J2 USB_B_Micro, J3 L834-1G1T-91, J4 105162-0001, J5 Conn_ARM_JTAG_SWD_10, J6 Conn_ARM_JTAG_SWD_10, P1 CONN_02x18, P10 CONN_01X01, P11 CONN_01X01, P13 CONN_01X01, P2 CONN_01x08, P3 CONN_01x08, P4 CONN_01x08, P5 CONN_01x10, P6 CONN_01x08, P7 CONN_01x08, P8 CONN_01X01, SW1 RESET, U1 STM32H730ZBT6, U10 S27KL0641DABHI020, U12 AP2161W, U2 IS25LP032D-JBLE-TR, U3 TPS62162DSG, U4 TPS62163DSG, U5 MAX40200AUK, U6 MAX40200AUK, U7 STM32F048G6Ux, U8 MAX40200AUK, U9 LAN8742A, Y1 32.768K, Y2 8M, Y3 25M

Commit message: Prepare for send to PCBWay
Signed-off-by: Martin Ribelotta <martinribelotta@gmail.com>
Parts:
- moved JP1 43.8 mm to (159.7, 102.5), turned to 180 degrees
- moved C41 7.81 mm to (116.5, 80.0)
- moved D3 4.55 mm to (116.6, 74.9), turned to 0 degrees
- moved LOGO1 2.68 mm to (153.8, 81.8)
- moved R5 2.36 mm to (159.8, 96.7)
- moved R26 1.23 mm to (116.6, 76.5), turned to 180 degrees
- moved C1 0.76 mm to (163.2, 100.5)
- moved C4 0.76 mm to (163.2, 98.9)
- moved C13 0.72 mm to (180.0, 105.1)
- moved R24 0.21 mm to (131.1, 98.0)
- moved G1 0.15 mm to (144.1, 76.6)
Connections:
- J3 pad 13: GND -> Net-(J3-Pad13)
- J3 pad 14: Net-(J3-Pad14) -> /Ethernet/LED1
- R24 pad 1: /Ethernet/LED1 -> GND
- R24 pad 2: Net-(J3-Pad14) -> Net-(J3-Pad13)
- R3 pad 1: +3V3 -> GND
Routing:
- net /BOOT0: track 51.1 -> 8.89 mm, vias 2 -> 0
- net Net-(J3-Pad14): track 22.7 -> 0.00 mm
- net /Ethernet/LED1: track 12.9 -> 35.2 mm
- net Net-(J3-Pad13): track 0.00 -> 19.8 mm
- net +3V3: track 106.8 -> 117.0 mm, vias 38 -> 36
- net /~RST: track 136.6 -> 142.8 mm
- net +5V: track 152.4 -> 148.6 mm
- net /Debug/DBG_SWCK: track 13.9 -> 17.3 mm
- net Net-(D3-Pad2): track 3.82 -> 1.60 mm
- net /53(SS): track 37.3 -> 39.4 mm
- net /52(SCK): track 34.4 -> 36.5 mm
- net /51(MOSI): track 34.9 -> 36.9 mm
- net /50(MISO): track 31.5 -> 33.2 mm
- net /CANRX: track 63.2 -> 61.9 mm
- net GND: track 176.6 -> 177.6 mm, vias 71 -> 72
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- added copper zone on In2.Cu, net Net-(C33-Pad1)
- removed copper zone on B.Cu, net Net-(C33-Pad1)
Other:
- board text added: "CM0 BOOT"
- board text added: "CM0 SWD"
- board text added: "CM7 BOOT"
- board text added: "CM7 SWD"
- board text added: "Copyright © 2021 Martin Ribelotta <martinribelotta@gmail.com> MIT License"
