File: USB-OTG.sch (KiCad schematic (older format))
At the start: 4 parts, among them J1 USB_C_Receptacle_USB2.0

Commit message: Replace non stocked components.
 - Redesign 5V/3.3V using TPS6216xDSGT
 - Use bigger crystal (move to 5031 case)
 - Change some components parts

Signed-off-by: Martin Ribelotta <martinribelotta@gmail.com>
Parts:
- D1: DESCRIPTION (none) -> SP0502BAHT
- J1: DESCRIPTION (none) -> USB C Receptacle Amphenol 12401610E4-2A
- R1, R2: DESCRIPTION (none) -> Resistor 1.5K 0603
Changed lines of the file:
@@
 F 2 "Package_TO_SOT_SMD:SOT-23" H 3975 3450 50  0001 L CNN
 F 3 "http://www.littelfuse.com/~/media/files/littelfuse/technical%20resources/documents/data%20sheets/sp05xxba.pdf" H 3875 3625 50  0001 C CNN
+F 4 "SP0502BAHT" H 3750 3500 50  0001 C CNN "DESCRIPTION"
 	1    3750 3500
 	1    0    0    -1
@@
 F 2 "footprints:USB_C_Receptacle_Amphenol_12401610E4-2A" H 2700 3100 50  0001 C CNN
 F 3 "https://www.usb.org/sites/default/files/documents/usb_type-c.zip" H 2700 3100 50  0001 C CNN
+F 4 "USB C Receptacle Amphenol 12401610E4-2A" H 2550 3100 50  0001 C CNN "DESCRIPTION"
 	1    2550 3100
 	1    0    0    -1
@@
 F 2 "Resistor_SMD:R_0603_1608Metric" H 3600 2700 50  0001 C CNN
 F 3 "~" H 3600 2700 50  0001 C CNN
+F 4 "Resistor 1.5K 0603" H 3600 2700 50  0001 C CNN "DESCRIPTION"
 	1    3600 2700
 	0    1    1    0
@@
 F 2 "Resistor_SMD:R_0603_1608Metric" H 3600 2800 50  0001 C CNN
 F 3 "~" H 3600 2800 50  0001 C CNN
+F 4 "Resistor 1.5K 0603" H 3600 2800 50  0001 C CNN "DESCRIPTION"
 	1    3600 2800
 	0    1    -1   0

Commit message: Add new BOM to octopart
TODO: PSRAM is not recognized by Octopart but is available in LCSC

Signed-off-by: Martin Ribelotta <martinribelotta@gmail.com>
Parts:
- D1: MANUFACTURER (none) -> Littlelfuse; MANUFACTURER_PART_NUMBER (none) -> SP0502BAHTG
- J1: MANUFACTURER (none) -> Ampenol; MANUFACTURER_PART_NUMBER (none) -> 12401610E4-2A
- R1, R2: MANUFACTURER (none) -> Yageo; MANUFACTURER_PART_NUMBER (none) -> RC0603JR-071K5L
Changed lines of the file:
@@
 F 3 "http://www.littelfuse.com/~/media/files/littelfuse/technical%20resources/documents/data%20sheets/sp05xxba.pdf" H 3875 3625 50  0001 C CNN
 F 4 "SP0502BAHT" H 3750 3500 50  0001 C CNN "DESCRIPTION"
+F 5 "Littlelfuse" H 3750 3500 50  0001 C CNN "MANUFACTURER"
+F 6 "SP0502BAHTG" H 3750 3500 50  0001 C CNN "MANUFACTURER_PART_NUMBER"
 	1    3750 3500
 	1    0    0    -1
@@
 F 3 "https://www.usb.org/sites/default/files/documents/usb_type-c.zip" H 2700 3100 50  0001 C CNN
 F 4 "USB C Receptacle Amphenol 12401610E4-2A" H 2550 3100 50  0001 C CNN "DESCRIPTION"
+F 5 "Ampenol" H 2550 3100 50  0001 C CNN "MANUFACTURER"
+F 6 "12401610E4-2A" H 2550 3100 50  0001 C CNN "MANUFACTURER_PART_NUMBER"
 	1    2550 3100
 	1    0    0    -1
@@
 F 3 "~" H 3600 2700 50  0001 C CNN
 F 4 "Resistor 1.5K 0603" H 3600 2700 50  0001 C CNN "DESCRIPTION"
+F 5 "Yageo" H 3600 2700 50  0001 C CNN "MANUFACTURER"
+F 6 "RC0603JR-071K5L" H 3600 2700 50  0001 C CNN "MANUFACTURER_PART_NUMBER"
 	1    3600 2700
 	0    1    1    0
@@
 F 3 "~" H 3600 2800 50  0001 C CNN
 F 4 "Resistor 1.5K 0603" H 3600 2800 50  0001 C CNN "DESCRIPTION"
+F 5 "Yageo" H 3600 2800 50  0001 C CNN "MANUFACTURER"
+F 6 "RC0603JR-071K5L" H 3600 2800 50  0001 C CNN "MANUFACTURER_PART_NUMBER"
 	1    3600 2800
 	0    1    -1   0
