File: h730duino.sch (KiCad schematic (older format))
At the start: 74 parts, among them J4 105162-0001, P1 CONN_02x18, P10 CONN_01X01, P11 CONN_01X01, P13 CONN_01X01, P2 CONN_01x08, P3 CONN_01x08, P4 CONN_01x08, P5 CONN_01x10, P6 CONN_01x08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

Commit message: Prepare for send to PCBWay
Signed-off-by: Martin Ribelotta <martinribelotta@gmail.com>
Parts:
- C14, C15: DESCRIPTION Capacitor 100n 0603 -> Capacitor 2.2u 0603
- D3, D4: DESCRIPTION Led SMD 0603 red -> RED Led SMD 0603
- P1: DESCRIPTION (none) -> Female pin shocket 02x18 2.54mm; MANUFACTURER Oupiin -> Oupin
- P2, P3, P4, P6, P7: DESCRIPTION (none) -> Female pin shocket 01x08 2.54mm
- P5: DESCRIPTION (none) -> Female pin shocket 01x10 2.54mm
- R11, R20, R27, R28, R29, R30, R31, R5: DESCRIPTION Resistor 1.5K 0603 -> Resistor 10K 0603
- SW1: DESCRIPTION (none) -> PTS645VL58-2 LFS
- U1: MANUFACTURER ST -> STMicroelectronics
- U10: DESCRIPTION (none) -> S27KL0641DABHI020; MANUFACTURER (none) -> cypress; MANUFACTURER_PART_NUMBER (none) -> S27KL0641DABHI020
- U12: DESCRIPTION (none) -> AP2161W
- U2: DESCRIPTION W25Q32JVSS -> IS25LP032D-JBLE-TR
- U3: DESCRIPTION (none) -> TPS62162DSG
- U4: DESCRIPTION (none) -> TPS62163DSG
- Y2: MANUFACTURER Abracon -> Abracom
Changed lines of the file:
@@
 F 4 "Oupin" H 14400 1650 50  0001 C CNN "MANUFACTURER"
 F 5 "2044-1X08G00SA" H 14400 1650 50  0001 C CNN "MANUFACTURER_PART_NUMBER"
+F 6 "Female pin shocket 01x08 2.54mm" H 14400 1650 50  0001 C CNN "DESCRIPTION"
 	1    14400 1650
 	1    0    0    -1
@@
 F 4 "Oupin" H 14800 1550 50  0001 C CNN "MANUFACTURER"
 F 5 "2044-1X10G00SA" H 14800 1550 50  0001 C CNN "MANUFACTURER_PART_NUMBER"
+F 6 "Female pin shocket 01x10 2.54mm" H 14800 1550 50  0001 C CNN "DESCRIPTION"
 	1    14800 1550
 	-1   0    0    -1
@@
 F 4 "Oupin" H 14400 2750 50  0001 C CNN "MANUFACTURER"
 F 5 "2044-1X08G00SA" H 14400 2750 50  0001 C CNN "MANUFACTURER_PART_NUMBER"
+F 6 "Female pin shocket 01x08 2.54mm" H 14400 2750 50  0001 C CNN "DESCRIPTION"
 	1    14400 2750
 	1    0    0    -1
@@
 F 4 "Oupin" H 14400 3700 50  0001 C CNN "MANUFACTURER"
 F 5 "2044-1X08G00SA" H 14400 3700 50  0001 C CNN "MANUFACTURER_PART_NUMBER"
+F 6 "Female pin shocket 01x08 2.54mm" H 14400 3700 50  0001 C CNN "DESCRIPTION"
 	1    14400 3700
 	1    0    0    -1
@@
 F 4 "Oupin" H 14800 3700 50  0001 C CNN "MANUFACTURER"
 F 5 "2044-1X08G00SA" H 14800 3700 50  0001 C CNN "MANUFACTURER_PART_NUMBER"
+F 6 "Female pin shocket 01x08 2.54mm" H 14800 3700 50  0001 C CNN "DESCRIPTION"
 	1    14800 3700
 	-1   0    0    -1
@@
 F 2 "Socket_Arduino_Mega:Socket_Strip_Arduino_2x18" H 14550 4000 50  0001 C CNN
 F 3 "" H 14550 4000 50  0000 C CNN
-F 4 "Oupiin" H 14550 5050 50  0001 C CNN "MANUFACTURER"
+F 4 "Oupin" H 14550 5050 50  0001 C CNN "MANUFACTURER"
 F 5 "2044-2X18G00SA" H 14550 5050 50  0001 C CNN "MANUFACTURER_PART_NUMBER"
+F 6 "Female pin shocket 02x18 2.54mm" H 14550 5050 50  0001 C CNN "DESCRIPTION"
 	1    14550 5050
 	0    -1   1    0
@@
 F 3 "~" H 1050 1400 50  0001 C CNN
 F 4 "Crystal 8MHz 3215" H 1050 1400 50  0001 C CNN "DESCRIPTION"
-F 5 "Abracon" H 1050 1400 50  0001 C CNN "MANUFACTURER"
+F 5 "Abracom" H 1050 1400 50  0001 C CNN "MANUFACTURER"
 F 6 "ABM7-8.000MHZ-D2Y-T" H 1050 1400 50  0001 C CNN "MANUFACTURER_PART_NUMBER"
 	1    1050 1400
@@
 F 2 "Capacitor_SMD:C_0603_1608Metric" H 3600 2850 50  0001 C CNN
 F 3 "~" H 3600 2850 50  0001 C CNN
-F 4 "Capacitor 100n 0603" H 3600 2850 50  0001 C CNN "DESCRIPTION"
+F 4 "Capacitor 2.2u 0603" H 3600 2850 50  0001 C CNN "DESCRIPTION"
 F 5 "CC0603ZRY5V6BB225" H 3600 2850 50  0001 C CNN "MANUFACTURER_PART_NUMBER"
 F 6 "Yageo" H 3600 2850 50  0001 C CNN "MANUFACTURER"
@@
 F 2 "Capacitor_SMD:C_0603_1608Metric" H 4000 2850 50  0001 C CNN
 F 3 "~" H 4000 2850 50  0001 C CNN
-F 4 "Capacitor 100n 0603" H 4000 2850 50  0001 C CNN "DESCRIPTION"
+F 4 "Capacitor 2.2u 0603" H 4000 2850 50  0001 C CNN "DESCRIPTION"
 F 5 "CC0603ZRY5V6BB225" H 4000 2850 50  0001 C CNN "MANUFACTURER_PART_NUMBER"
 F 6 "Yageo" H 4000 2850 50  0001 C CNN "MANUFACTURER"
@@
 F 2 "LED_SMD:LED_0603_1608Metric" V 9900 4050 50  0001 C CNN
 F 3 "~" V 9900 4050 50  0001 C CNN
-F 4 "Led SMD 0603 red" H 9900 4050 50  0001 C CNN "DESCRIPTION"
+F 4 "RED Led SMD 0603" H 9900 4050 50  0001 C CNN "DESCRIPTION"
 F 5 "Osram" H 9900 4050 50  0001 C CNN "MANUFACTURER"
 F 6 "LS Q976-NR-1" H 9900 4050 50  0001 C CNN "MANUFACTURER_PART_NUMBER"
@@
 F 4 "C&K" H 1000 2600 50  0001 C CNN "MANUFACTURER"
 F 5 "PTS645VL58-2 LFS" H 1000 2600 50  0001 C CNN "MANUFACTURER_PART_NUMBER"
+F 6 "PTS645VL58-2 LFS" H 1000 2600 50  0001 C CNN "DESCRIPTION"
 	1    1000 2600
 	1    0    0    -1
@@
 F 2 "LED_SMD:LED_0603_1608Metric" V 9650 4050 50  0001 C CNN
 F 3 "~" V 9650 4050 50  0001 C CNN
-F 4 "Led SMD 0603 red" H 9650 4050 50  0001 C CNN "DESCRIPTION"
+F 4 "RED Led SMD 0603" H 9650 4050 50  0001 C CNN "DESCRIPTION"
 F 5 "Osram" H 9650 4050 50  0001 C CNN "MANUFACTURER"
 F 6 "LS Q976-NR-1" H 9650 4050 50  0001 C CNN "MANUFACTURER_PART_NUMBER"
@@
 F 2 "Resistor_SMD:R_0603_1608Metric" H 850 2100 50  0001 C CNN
 F 3 "~" H 850 2100 50  0001 C CNN
-F 4 "Resistor 1.5K 0603" H 850 2100 50  0001 C CNN "DESCRIPTION"
+F 4 "Resistor 10K 0603" H 850 2100 50  0001 C CNN "DESCRIPTION"
 F 5 "Yageo" H 850 2100 50  0001 C CNN "MANUFACTURER"
 F 6 "RC0603FR-0710KL" H 850 2100 50  0001 C CNN "MANUFACTURER_PART_NUMBER"
@@
 F 3 "" H 2100 500 60  0000 C CNN
 F 4 "STM32H730ZBT6" H 1800 900 50  0001 C CNN "DESCRIPTION"
-F 5 "ST" H 1800 900 50  0001 C CNN "MANUFACTURER"
+F 5 "STMicroelectronics" H 1800 900 50  0001 C CNN "MANUFACTURER"
 F 6 "STM32H730ZBT6" H 1800 900 50  0001 C CNN "MANUFACTURER_PART_NUMBER"
 	3    1800 900
@@
 F 3 "" H 5600 950 60  0000 C CNN
 F 4 "STM32H730ZBT6" H 5300 1350 50  0001 C CNN "DESCRIPTION"
-F 5 "ST" H 5300 1350 50  0001 C CNN "MANUFACTURER"
+F 5 "STMicroelectronics" H 5300 1350 50  0001 C CNN "MANUFACTURER"
 F 6 "STM32H730ZBT6" H 5300 1350 50  0001 C CNN "MANUFACTURER_PART_NUMBER"
 	1    5300 1350
@@
 F 3 "" H 2050 4300 60  0000 C CNN
 F 4 "STM32H730ZBT6" H 1750 4700 50  0001 C CNN "DESCRIPTION"
-F 5 "ST" H 1750 4700 50  0001 C CNN "MANUFACTURER"
+F 5 "STMicroelectronics" H 1750 4700 50  0001 C CNN "MANUFACTURER"
 F 6 "STM32H730ZBT6" H 1750 4700 50  0001 C CNN "MANUFACTURER_PART_NUMBER"
 	2    1750 4700
@@
 F 2 "footprints:SOIC-8_5.23x5.23mm_P1.27mm" H 11350 6050 50  0001 C CNN
 F 3 "http://www.winbond.com/resource-files/w25q32jv%20revg%2003272018%20plus.pdf" H 11350 6050 50  0001 C CNN
-F 4 "W25Q32JVSS" H 11350 6050 50  0001 C CNN "DESCRIPTION"
+F 4 "IS25LP032D-JBLE-TR" H 11350 6050 50  0001 C CNN "DESCRIPTION"
 F 5 "ISSI" H 11350 6050 50  0001 C CNN "MANUFACTURER"
 F 6 "IS25LP032D-JBLE-TR" H 11350 6050 50  0001 C CNN "MANUFACTURER_PART_NUMBER"
@@
 F 4 "Oupin" H 14800 2750 50  0001 C CNN "MANUFACTURER"
 F 5 "2044-1X08G00SA" H 14800 2750 50  0001 C CNN "MANUFACTURER_PART_NUMBER"
+F 6 "Female pin shocket 01x08 2.54mm" H 14800 2750 50  0001 C CNN "DESCRIPTION"
 	1    14800 2750
 	-1   0    0    -1
@@
 F 4 "TI" H 10000 1450 50  0001 C CNN "MANUFACTURER"
 F 5 "TPS62163DSG" H 10000 1450 50  0001 C CNN "MANUFACTURER_PART_NUMBER"
+F 6 "TPS62163DSG" H 10000 1450 50  0001 C CNN "DESCRIPTION"
 	1    10000 1450
 	1    0    0    -1
@@
 F 4 "TI" H 10000 2500 50  0001 C CNN "MANUFACTURER"
 F 5 "TPS62162DSG" H 10000 2500 50  0001 C CNN "MANUFACTURER_PART_NUMBER"
+F 6 "TPS62162DSG" H 10000 2500 50  0001 C CNN "DESCRIPTION"
 	1    10000 2500
 	1    0    0    -1
@@
 F 2 "Resistor_SMD:R_0603_1608Metric" H 1500 2600 50  0001 C CNN
 F 3 "~" H 1500 2600 50  0001 C CNN
-F 4 "Resistor 1.5K 0603" H 1500 2600 50  0001 C CNN "DESCRIPTION"
+F 4 "Resistor 10K 0603" H 1500 2600 50  0001 C CNN "DESCRIPTION"
 F 5 "Yageo" H 1500 2600 50  0001 C CNN "MANUFACTURER"
 F 6 "RC0603FR-0710KL" H 1500 2600 50  0001 C CNN "MANUFACTURER_PART_NUMBER"
@@
 F 2 "Resistor_SMD:R_0603_1608Metric" H 12150 8650 50  0001 C CNN
 F 3 "~" H 12150 8650 50  0001 C CNN
-F 4 "Resistor 1.5K 0603" H 12150 8650 50  0001 C CNN "DESCRIPTION"
+F 4 "Resistor 10K 0603" H 12150 8650 50  0001 C CNN "DESCRIPTION"
 F 5 "Yageo" H 12150 8650 50  0001 C CNN "MANUFACTURER"
 F 6 "RC0603FR-0710KL" H 12150 8650 50  0001 C CNN "MANUFACTURER_PART_NUMBER"
@@
 F 2 "Resistor_SMD:R_0603_1608Metric" H 12050 8650 50  0001 C CNN
 F 3 "~" H 12050 8650 50  0001 C CNN
-F 4 "Resistor 1.5K 0603" H 12050 8650 50  0001 C CNN "DESCRIPTION"
+F 4 "Resistor 10K 0603" H 12050 8650 50  0001 C CNN "DESCRIPTION"
 F 5 "Yageo" H 12050 8650 50  0001 C CNN "MANUFACTURER"
 F 6 "RC0603FR-0710KL" H 12050 8650 50  0001 C CNN "MANUFACTURER_PART_NUMBER"
@@
 F 2 "Resistor_SMD:R_0603_1608Metric" H 11950 8650 50  0001 C CNN
 F 3 "~" H 11950 8650 50  0001 C CNN
-F 4 "Resistor 1.5K 0603" H 11950 8650 50  0001 C CNN "DESCRIPTION"
+F 4 "Resistor 10K 0603" H 11950 8650 50  0001 C CNN "DESCRIPTION"
 F 5 "Yageo" H 11950 8650 50  0001 C CNN "MANUFACTURER"
 F 6 "RC0603FR-0710KL" H 11950 8650 50  0001 C CNN "MANUFACTURER_PART_NUMBER"
@@
 F 2 "Resistor_SMD:R_0603_1608Metric" H 11850 8650 50  0001 C CNN
 F 3 "~" H 11850 8650 50  0001 C CNN
-F 4 "Resistor 1.5K 0603" H 11850 8650 50  0001 C CNN "DESCRIPTION"
+F 4 "Resistor 10K 0603" H 11850 8650 50  0001 C CNN "DESCRIPTION"
 F 5 "Yageo" H 11850 8650 50  0001 C CNN "MANUFACTURER"
 F 6 "RC0603FR-0710KL" H 11850 8650 50  0001 C CNN "MANUFACTURER_PART_NUMBER"
@@
 F 2 "Resistor_SMD:R_0603_1608Metric" H 11750 8650 50  0001 C CNN
 F 3 "~" H 11750 8650 50  0001 C CNN
-F 4 "Resistor 1.5K 0603" H 11750 8650 50  0001 C CNN "DESCRIPTION"
+F 4 "Resistor 10K 0603" H 11750 8650 50  0001 C CNN "DESCRIPTION"
 F 5 "Yageo" H 11750 8650 50  0001 C CNN "MANUFACTURER"
 F 6 "RC0603FR-0710KL" H 11750 8650 50  0001 C CNN "MANUFACTURER_PART_NUMBER"
@@
 F 4 "Diodes" H 12300 3600 50  0001 C CNN "MANUFACTURER"
 F 5 "AP2161W" H 12300 3600 50  0001 C CNN "MANUFACTURER_PART_NUMBER"
+F 6 "AP2161W" H 12300 3600 50  0001 C CNN "DESCRIPTION"
 	1    12300 3600
 	-1   0    0    -1
@@
 F 2 "footprints:S27KL0641DABHI020" H 7550 6340 60  0001 C CNN
 F 3 "" H 7400 7400 60  0000 C CNN
+F 4 "cypress" H 6750 6000 50  0001 C CNN "MANUFACTURER"
+F 5 "S27KL0641DABHI020" H 6750 6000 50  0001 C CNN "MANUFACTURER_PART_NUMBER"
+F 6 "S27KL0641DABHI020" H 6750 6000 50  0001 C CNN "DESCRIPTION"
 	1    6750 6000
 	1    0    0    -1
@@
 F 2 "Resistor_SMD:R_0603_1608Metric" H 6000 5800 50  0001 C CNN
 F 3 "~" H 6000 5800 50  0001 C CNN
-F 4 "Resistor 1.5K 0603" H 6000 5800 50  0001 C CNN "DESCRIPTION"
+F 4 "Resistor 10K 0603" H 6000 5800 50  0001 C CNN "DESCRIPTION"
 F 5 "Yageo" H 6000 5800 50  0001 C CNN "MANUFACTURER"
 F 6 "RC0603FR-0710KL" H 6000 5800 50  0001 C CNN "MANUFACTURER_PART_NUMBER"

Commit message: Fix 1V8 issue and OSPI pinout
Signed-off-by: Martin Ribelotta <martinribelotta@gmail.com>
Connections:
- net OCTOSPIM_P1_IO0: now also U10.E3 (DQ5); no longer U10.E2 (DQ6)
- net OCTOSPIM_P1_IO1: now also U10.D5 (DQ4); no longer U10.E1 (DQ7)
- net OCTOSPIM_P1_IO2: now also U10.E2 (DQ6); no longer U10.E3 (DQ5)
- net OCTOSPIM_P1_IO3: now also U10.E1 (DQ7); no longer U10.D5 (DQ4)
Changed lines of the file:
@@
 Text Label 6750 6450 2    50   ~ 0
 OCTOSPIM_P2_IO3
-Text Label 6750 6550 2    50   ~ 0
-OCTOSPIM_P1_IO3
-Text Label 6750 6650 2    50   ~ 0
-OCTOSPIM_P1_IO2
-Text Label 6750 6750 2    50   ~ 0
-OCTOSPIM_P1_IO0
-Text Label 6750 6850 2    50   ~ 0
-OCTOSPIM_P1_IO1
 Text Label 3950 5900 0    50   ~ 0
 OCTOSPIM_P2_DQS
@@
 	1    0    0    -1
 $EndComp
+Text Label 6750 6550 2    50   ~ 0
+OCTOSPIM_P1_IO1
+Text Label 6750 6650 2    50   ~ 0
+OCTOSPIM_P1_IO0
+Text Label 6750 6750 2    50   ~ 0
+OCTOSPIM_P1_IO2
+Text Label 6750 6850 2    50   ~ 0
+OCTOSPIM_P1_IO3
 $EndSCHEMATC

Commit message: REally fix HyperRAM connection.
Additionally:
 - Fix PTH on ETH connector
 - Move USB-C to the left

Signed-off-by: Martin Ribelotta <martinribelotta@gmail.com>
Parts:
- LOGO1: footprint Symbol:OSHW-Logo_5.7x6mm_SilkScreen -> Symbol:OSHW-Logo_7.5x8mm_SilkScreen
Connections:
- net GND: now also SW1.2; no longer SW1.1
- net OCTOSPIM_P1_IO0: now also U10.D5 (DQ4); no longer U10.E3 (DQ5)
- net OCTOSPIM_P1_IO1: now also U10.E3 (DQ5); no longer U10.D5 (DQ4)
- net ~RST: now also SW1.1; no longer SW1.2
Changed lines of the file:
@@
 F 6 "PTS645VL58-2 LFS" H 1000 2600 50  0001 C CNN "DESCRIPTION"
 	1    1000 2600
-	1    0    0    -1
+	-1   0    0    -1
 $EndComp
 $Sheet
@@
 F 0 "LOGO1" H 12200 10575 50  0001 C CNN
 F 1 "Logo_Open_Hardware_Small" H 12200 10075 50  0001 C CNN
-F 2 "Symbol:OSHW-Logo_5.7x6mm_SilkScreen" H 12200 10300 50  0001 C CNN
+F 2 "Symbol:OSHW-Logo_7.5x8mm_SilkScreen" H 12200 10300 50  0001 C CNN
 F 3 "~" H 12200 10300 50  0001 C CNN
 	1    12200 10300
@@
 	1    0    0    -1
 $EndComp
+Text Label 6750 6650 2    50   ~ 0
+OCTOSPIM_P1_IO1
 Text Label 6750 6550 2    50   ~ 0
-OCTOSPIM_P1_IO1
-Text Label 6750 6650 2    50   ~ 0
 OCTOSPIM_P1_IO0
 Text Label 6750 6750 2    50   ~ 0

Commit message: Add QR of project URL
Signed-off-by: Martin Ribelotta <martinribelotta@gmail.com>
Parts:
- removed U8: MAX40200AUK, Package_TO_SOT_SMD:SOT-23-5, symbol Analog_Switch:MAX40200AUK
- added J2: Conn_02x03_Odd_Even, Connector_PinHeader_2.54mm:PinHeader_2x03_P2.54mm_Horizontal, symbol Connector_Generic:Conn_02x03_Odd_Even
Connections:
- net GND: now also J2.2 (Pin_2)
- net OCTOSPIM_P1_IO0: now also U10.D3 (DQ0); no longer U10.D5 (DQ4)
- net OCTOSPIM_P1_IO1: now also U10.D2 (DQ1); no longer U10.E3 (DQ5)
- net OCTOSPIM_P1_IO2: now also U10.C4 (DQ2); no longer U10.E2 (DQ6)
- net OCTOSPIM_P1_IO3: now also U10.D4 (DQ3); no longer U10.E1 (DQ7)
- net OCTOSPIM_P2_IO0: now also U10.D5 (DQ4); no longer U10.D3 (DQ0)
- net OCTOSPIM_P2_IO1: now also U10.E3 (DQ5); no longer U10.D2 (DQ1)
- net OCTOSPIM_P2_IO2: now also U10.E2 (DQ6); no longer U10.C4 (DQ2)
- net OCTOSPIM_P2_IO3: now also U10.E1 (DQ7); no longer U10.D4 (DQ3)
- net SWCLK: now also J2.6 (Pin_6)
- net SWDIO: now also J2.4 (Pin_4)
- net USART1_RX: now also J2.3 (Pin_3)
- net USART1_TX: now also J2.5 (Pin_5)
- net ~RST: now also J2.1 (Pin_1)
Changed lines of the file:
@@
 $Descr A3 16535 11693
 encoding utf-8
-Sheet 1 4
+Sheet 1 3
 Title ""
 Date "mar. 31 mars 2015"
@@
 	-1   0    0    -1
 $EndComp
-$Sheet
-S 12700 6950 750  800
-U 60158DDC
-F0 "Debug" 50
-F1 "debugger.sch" 50
-F2 "SWCK" O L 12700 7500 50
-F3 "SWDIO" B L 12700 7400 50
-F4 "UART_TX" O L 12700 7050 50
-F5 "UART_RX" I L 12700 7150 50
-F6 "~RESET_OUT" O L 12700 7300 50
-F7 "VBUS_DBG" O L 12700 7650 50
-$EndSheet
-Text Label 12600 7050 2    50   ~ 0
+Text Label 11350 4900 2    50   ~ 0
 USART1_RX
-Text Label 12600 7150 2    50   ~ 0
+Text Label 11350 5000 2    50   ~ 0
 USART1_TX
 Wire Wire Line
-	12700 7050 12600 7050
-Wire Wire Line
-	12600 7150 12700 7150
-Text Label 12600 7300 2    50   ~ 0
+	11450 4800 11350 4800
+Wire Wire Line
+	11350 4900 11450 4900
+Text Label 11350 4800 2    50   ~ 0
 ~RST
 Wire Wire Line
-	12600 7300 12700 7300
-Wire Wire Line
-	12800 2750 12800 1950
-Wire Wire Line
-	12700 2750 12800 2750
-Wire Wire Line
-	11900 2950 11900 2750
-$Comp
-L power:GND #PWR0103
-U 1 1 601E2B1C
-P 12300 3150
-F 0 "#PWR0103" H 12300 2900 50  0001 C CNN
-F 1 "GND" V 12300 2950 50  0000 C CNN
-F 2 "" H 12300 3150 50  0000 C CNN
-F 3 "" H 12300 3150 50  0000 C CNN
-	1    12300 3150
-	0    -1   -1   0
-$EndComp
-Connection ~ 11900 2750
-$Comp
-L Analog_Switch:MAX40200AUK U8
-U 1 1 601E2B23
-P 12300 2850
-F 0 "U8" H 12300 3217 50  0000 C CNN
-F 1 "MAX40200AUK" H 12300 3126 50  0000 C CNN
-F 2 "Package_TO_SOT_SMD:SOT-23-5" H 12300 3350 50  0001 C CNN
-F 3 "https://datasheets.maximintegrated.com/en/ds/MAX40200.pdf" H 12300 3350 50  0001 C CNN
-F 4 "MAX40200AUK" H 12300 2850 50  0001 C CNN "DESCRIPTION"
-F 5 "Maxim" H 12300 2850 50  0001 C CNN "MANUFACTURER"
-F 6 "MAX40200AUK" H 12300 2850 50  0001 C CNN "MANUFACTURER_PART_NUMBER"
-	1    12300 2850
-	1    0    0    -1
-$EndComp
-Text Label 11500 2750 0    50   ~ 0
-DBG_VBUS
-Text Label 12600 7650 2    50   ~ 0
-DBG_VBUS
-Wire Wire Line
-	12600 7650 12700 7650
-Wire Wire Line
-	12700 7400 12600 7400
-Wire Wire Line
-	12600 7500 12700 7500
-Text Label 12600 7500 2    50   ~ 0
+	12050 5000 11950 5000
+Wire Wire Line
+	11950 4800 12250 4800
+Wire Wire Line
+	12050 4900 11950 4900
+Text Label 12050 5000 0    50   ~ 0
 SWCLK
-Text Label 12600 7400 2    50   ~ 0
+Text Label 12050 4900 0    50   ~ 0
 SWDIO
 Text Label 13450 1550 2    50   ~ 0
@@
 $EndComp
 Wire Wire Line
-	12800 2750 12800 3500
-Wire Wire Line
 	12800 3500 12700 3500
-Connection ~ 12800 2750
 Wire Wire Line
 	12700 3700 12700 4100
@@
 $EndComp
 Connection ~ 12800 1950
-Wire Wire Line
-	11500 2750 11900 2750
 $Comp
 L power:VBUS #PWR0107
@@
 U 1 1 6069A575
 P 12150 8650
-F 0 "R31" H 12200 8900 50  0000 R CNN
+F 0 "R31" V 12150 8950 50  0000 R CNN
 F 1 "10K" V 12100 8550 50  0000 R CNN
 F 2 "Resistor_SMD:R_0603_1608Metric" H 12150 8650 50  0001 C CNN
@@
 U 1 1 6069CA86
 P 12050 8650
-F 0 "R30" H 12100 8800 50  0000 R CNN
+F 0 "R30" V 12050 8950 50  0000 R CNN
 F 1 "10K" V 12000 8550 50  0000 R CNN
 F 2 "Resistor_SMD:R_0603_1608Metric" H 12050 8650 50  0001 C CNN
@@
 U 1 1 6069CCE5
 P 11950 8650
-F 0 "R29" H 12000 8900 50  0000 R CNN
+F 0 "R29" V 11950 8950 50  0000 R CNN
 F 1 "10K" V 11900 8550 50  0000 R CNN
 F 2 "Resistor_SMD:R_0603_1608Metric" H 11950 8650 50  0001 C CNN
@@
 U 1 1 6069D01E
 P 11850 8650
-F 0 "R28" H 11900 8800 50  0000 R CNN
+F 0 "R28" V 11850 8950 50  0000 R CNN
 F 1 "10K" V 11800 8550 50  0000 R CNN
 F 2 "Resistor_SMD:R_0603_1608Metric" H 11850 8650 50  0001 C CNN
@@
 U 1 1 6069D327
 P 11750 8650
-F 0 "R27" H 11700 8900 50  0000 L CNN
+F 0 "R27" V 11750 8800 50  0000 L CNN
 F 1 "10K" V 11700 8400 50  0000 L CNN
 F 2 "Resistor_SMD:R_0603_1608Metric" H 11750 8650 50  0001 C CNN
@@
 Text Label 6750 7250 2    50   ~ 0
 OCTOSPIM_P2_CLK
-Text Label 6750 6150 2    50   ~ 0
+Text Label 6750 6550 2    50   ~ 0
 OCTOSPIM_P2_IO0
-Text Label 6750 6250 2    50   ~ 0
+Text Label 6750 6650 2    50   ~ 0
 OCTOSPIM_P2_IO1
-Text Label 6750 6350 2    50   ~ 0
+Text Label 6750 6750 2    50   ~ 0
 OCTOSPIM_P2_IO2
-Text Label 6750 6450 2    50   ~ 0
+Text Label 6750 6850 2    50   ~ 0
 OCTOSPIM_P2_IO3
 Text Label 3950 5900 0    50   ~ 0
@@
 	1    0    0    -1
 $EndComp
-Text Label 6750 6650 2    50   ~ 0
+Text Label 6750 6250 2    50   ~ 0
 OCTOSPIM_P1_IO1
-Text Label 6750 6550 2    50   ~ 0
+Text Label 6750 6150 2    50   ~ 0
 OCTOSPIM_P1_IO0
-Text Label 6750 6750 2    50   ~ 0
+Text Label 6750 6350 2    50   ~ 0
 OCTOSPIM_P1_IO2
-Text Label 6750 6850 2    50   ~ 0
+Text Label 6750 6450 2    50   ~ 0
 OCTOSPIM_P1_IO3
+Wire Wire Line
+	12800 1950 12800 3500
+$Comp
+L Connector_Generic:Conn_02x03_Odd_Even J2
+U 1 1 6113E92E
+P 11650 4900
+F 0 "J2" H 11700 5217 50  0000 C CNN
+F 1 "Conn_02x03_Odd_Even" H 11700 5126 50  0000 C CNN
+F 2 "Connector_PinHeader_2.54mm:PinHeader_2x03_P2.54mm_Horizontal" H 11650 4900 50  0001 C CNN
+F 3 "~" H 11650 4900 50  0001 C CNN
+	1    11650 4900
+	1    0    0    -1
+$EndComp
+$Comp
+L power:GND #PWR012
+U 1 1 611AE3AA
+P 12250 4800
+F 0 "#PWR012" H 12250 4550 50  0001 C CNN
+F 1 "GND" V 12255 4672 50  0000 R CNN
+F 2 "" H 12250 4800 50  0000 C CNN
+F 3 "" H 12250 4800 50  0000 C CNN
+	1    12250 4800
+	0    -1   -1   0
+$EndComp
+Wire Wire Line
+	11350 5000 11450 5000
 $EndSCHEMATC
